File: choc660/choc660.kicad_pcb (KiCad board)
At the start: 2 copper layers, 29.3 x 11.3 mm, 144 parts, among them SW1 SW_Push, SW10 SW_Push, SW11 SW_Push, SW12 SW_Push, SW13 SW_Push, SW14 SW_Push, SW15 SW_Push, SW16 SW_Push, SW17 SW_Push, SW18 SW_Push, SW19 SW_Push, SW2 SW_Push, SW20 SW_Push, SW21 SW_Push, SW22 SW_Push, SW23 SW_Push, SW24 SW_Push, SW25 SW_Push, SW26 SW_Push, SW27 SW_Push, SW28 SW_Push, SW29 SW_Push, SW3 SW_Push, SW30 SW_Push, SW31 SW_Push, SW32 SW_Push, SW33 SW_Push, SW34 SW_Push, SW35 SW_Push, SW36 SW_Push, SW37 SW_Push, SW38 SW_Push, SW39 SW_Push, SW4 SW_Push, SW40 SW_Push, SW41 SW_Push, SW42 SW_Push, SW43 SW_Push, SW44 SW_Push, SW45 SW_Push, SW46 SW_Push, SW47 SW_Push, SW48 SW_Push, SW49 SW_Push, SW5 SW_Push, SW50 SW_Push, SW51 SW_Push, SW52 SW_Push, SW53 SW_Push, SW54 SW_Push, SW55 SW_Push, SW56 SW_Push, SW57 SW_Push, SW58 SW_Push, SW59 SW_Push, SW6 SW_Push, SW60 SW_Push, SW61 SW_Push, SW62 SW_Push, SW63 SW_Push, SW64 SW_Push, SW65 SW_Push, SW66 SW_Push, SW67 SW_Push, SW68 SW_Push, SW7 SW_Push, SW8 SW_Push, SW9 SW_Push, U1 Elite-C

Commit message: place diodes
Parts:
- moved SW68 205.2 mm to (351.5, 113.0)
- moved S1 192.3 mm to (307.0, 133.5)
- moved S2 192.3 mm to (311.5, 99.5)
- moved S3 192.3 mm to (77.5, 150.5)
- moved S4 192.3 mm to (298.0, 150.5)
- moved S5 192.3 mm to (140.5, 167.5)
- moved S6 192.3 mm to (176.5, 167.5)
- moved S7 192.3 mm to (212.5, 167.5)
- moved SW1 192.3 mm to (68.5, 99.5)
- moved SW10 192.3 mm to (91.0, 167.5)
- moved SW11 192.3 mm to (104.5, 99.5)
- moved SW12 192.3 mm to (113.5, 116.5)
- moved SW13 192.3 mm to (118.0, 133.5)
- moved SW14 192.3 mm to (127.0, 150.5)
- moved SW15 192.3 mm to (113.5, 167.5)
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Other:
- outline, holes or cut-outs redrawn

Commit message: draw the rest of the owl?
Parts:
- removed S1, S2, S3, S4, S5, S6, S7: MX_stab, marbastlib-choc:STAB_choc_2u
- added D65: SOD-123, Diode_SMD:D_SOD-123, B.Cu at (61.7, 167.0)
- added SW65: SW_Push, marbastlib-choc:SW_choc_HS_1u, F.Cu at (70.7, 167.5)
- D1, D10, D11, D12, D13, D14, D15, D16, D17, D18, D19, D2, D20, D21, D22, D23, D24, D25, D26, D27, D28, D29, D3, D30, D31, D32, D33, D34, D35, D36, D37, D38, D39, D4, D40, D41, D42, D43, D44, D45, D46, D47, D48, D49, D5, D50, D51, D52, D53, D54, D55, D56, D57, D58, D59, D6, D60, D61, D62, D63, D64, D7, D8, D9: moved to B.Cu
- D66: renamed from D65; moved to B.Cu
- D67: renamed from D66; moved to B.Cu
- D68: renamed from D67; moved to B.Cu
- D69: renamed from D68; moved to B.Cu
- SW1, SW10, SW11, SW12, SW13, SW14, SW15, SW16, SW17, SW18, SW19, SW2, SW21, SW22, SW23, SW24, SW26, SW27, SW28, SW29, SW3, SW31, SW32, SW33, SW34, SW36, SW37, SW38, SW39, SW40, SW41, SW42, SW43, SW44, SW45, SW46, SW47, SW48, SW49, SW5, SW50, SW51, SW52, SW53, SW54, SW55, SW56, SW57, SW58, SW6, SW60, SW61, SW62, SW64, SW7, SW8, SW9: moved to F.Cu
- SW20, SW25, SW30, SW35, SW4, SW59, SW63: footprint marbastlib-choc:SW_choc_HS_1u -> marbastlib-choc:SW_choc_HS_1.5u; moved to F.Cu
- SW66: renamed from SW65; footprint marbastlib-choc:SW_choc_HS_1u -> marbastlib-choc:SW_choc_HS_1.5u; moved to F.Cu
- SW67: renamed from SW66; footprint marbastlib-choc:SW_choc_HS_1.5u -> marbastlib-choc:SW_choc_HS_1u; moved to F.Cu
- SW68: renamed from SW67; moved to F.Cu
- SW69: renamed from SW68; moved to F.Cu
- moved D69 298.8 mm to (61.7, 116.0)
- moved D68 298.8 mm to (61.7, 99.0)
- moved SW1 285.2 mm to (353.7, 99.5), turned to 0 degrees
- moved SW69 280.8 mm to (70.7, 116.5), turned to 0 degrees
- moved SW68 280.8 mm to (70.7, 99.5), turned to 0 degrees
- moved D60 280.8 mm to (79.7, 167.0)
- moved SW2 276.2 mm to (349.2, 116.5), turned to 0 degrees
- moved SW3 271.7 mm to (344.7, 133.5), turned to 0 degrees
- moved D1 267.2 mm to (344.7, 99.0)
- moved SW5 267.2 mm to (335.7, 167.5), turned to 0 degrees
- moved D64 262.8 mm to (79.7, 151.0)
- moved SW60 262.8 mm to (88.7, 167.5), turned to 0 degrees
- moved D2 258.2 mm to (340.2, 116.0)
- moved SW4 258.2 mm to (335.7, 150.5), turned to 0 degrees
- moved D3 253.7 mm to (335.7, 133.0)
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Connections:
- U1 pad 10: R0 -> R9
- U1 pad 11: R1 -> R8
- U1 pad 12: R2 -> R7
- U1 pad 13: R3 -> R6
- U1 pad 14: R4 -> R5
- U1 pad 15: R5 -> R4
- U1 pad 16: R6 -> R3
- U1 pad 17: R7 -> R2
- U1 pad 18: R8 -> R1
- U1 pad 19: R9 -> R0
Routing:
- net C0: track 0.00 -> 443.8 mm
- net C1: track 0.00 -> 418.3 mm
- net C2: track 0.00 -> 411.3 mm
- net R9: track 0.00 -> 407.9 mm
- net R7: track 0.00 -> 386.0 mm
- net R8: track 0.00 -> 375.2 mm
- net R5: track 0.00 -> 359.8 mm
- net C3: track 0.00 -> 358.5 mm
- net C4: track 0.00 -> 321.8 mm
- net R1: track 0.00 -> 314.6 mm
- net R6: track 0.00 -> 312.7 mm
- net R3: track 0.00 -> 303.9 mm
- net R0: track 0.00 -> 300.3 mm
- net C5: track 0.00 -> 299.0 mm
- net R4: track 0.00 -> 287.2 mm
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Other:
- board size 29.3 x 11.3 mm -> 305 x 86 mm

Commit message: use non-hotswap footprints, also i made this backwards
Parts:
- D1, D10, D11, D12, D13, D14, D15, D16, D17, D18, D19, D2, D20, D21, D22, D23, D24, D25, D26, D27, D28, D29, D3, D30, D31, D32, D33, D34, D35, D36, D37, D38, D39, D4, D40, D41, D42, D43, D44, D45, D46, D47, D48, D49, D5, D50, D51, D52, D53, D54, D55, D56, D57, D58, D59, D6, D60, D61, D62, D63, D64, D65, D66, D67, D68, D69, D7, D8, D9: moved to F.Cu
- SW1, SW10, SW11, SW12, SW13, SW14, SW15, SW16, SW17, SW18, SW19, SW21, SW22, SW23, SW24, SW26, SW27, SW28, SW29, SW31, SW32, SW33, SW34, SW36, SW37, SW38, SW39, SW40, SW41, SW42, SW43, SW44, SW45, SW46, SW47, SW48, SW49, SW5, SW50, SW51, SW52, SW53, SW54, SW55, SW56, SW57, SW58, SW6, SW60, SW61, SW62, SW64, SW65, SW67, SW68, SW69, SW7, SW8, SW9: footprint marbastlib-choc:SW_choc_HS_1u -> marbastlib-choc:SW_choc_1u; moved to B.Cu
- SW2, SW25, SW3, SW30, SW35, SW4, SW59, SW63, SW66: footprint marbastlib-choc:SW_choc_HS_1.5u -> marbastlib-choc:SW_choc_1.5u; moved to B.Cu
- SW20: footprint marbastlib-choc:SW_choc_HS_1.5u -> marbastlib-choc:SW_choc_1.25u; moved to B.Cu
- U1: moved to B.Cu
- moved D65 298.1 mm to (359.8, 167.0)
- moved D68 298.1 mm to (359.8, 99.0)
- moved D69 298.1 mm to (359.8, 116.0)
- moved SW1 285.9 mm to (67.8, 99.5), turned to 180 degrees
- moved SW65 280.1 mm to (350.8, 167.5), turned to 180 degrees
- moved SW68 280.1 mm to (350.8, 99.5), turned to 180 degrees
- moved SW69 280.1 mm to (350.8, 116.5), turned to 180 degrees
- moved SW2 276.9 mm to (72.3, 116.5), turned to 180 degrees
- moved D1 267.9 mm to (76.8, 99.0)
- moved SW3 267.9 mm to (76.8, 133.5), turned to 180 degrees
- moved D64 262.1 mm to (341.8, 150.0)
- moved D60 262.1 mm to (341.8, 167.0)
- moved D2 258.9 mm to (81.3, 116.0)
- moved D3 249.9 mm to (85.8, 133.0)
- moved SW4 249.9 mm to (85.8, 150.5), turned to 180 degrees
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Routing:
- net R7: track 386.0 -> 392.0 mm
- net Net-(D64-Pad2): track 2.91 -> 6.50 mm
- net Net-(D15-Pad2): track 2.91 -> 6.18 mm
- net Net-(D9-Pad2): track 2.91 -> 6.18 mm
- net Net-(D8-Pad2): track 2.91 -> 6.18 mm
- net Net-(D5-Pad2): track 2.91 -> 6.18 mm
- net Net-(D4-Pad2): track 2.91 -> 6.18 mm
- net Net-(D3-Pad2): track 2.91 -> 6.18 mm
- net Net-(D13-Pad2): track 2.91 -> 6.18 mm
- net Net-(D10-Pad2): track 2.91 -> 6.18 mm
- net Net-(D63-Pad2): track 2.91 -> 6.18 mm
- net Net-(D60-Pad2): track 2.91 -> 6.18 mm
- net Net-(D59-Pad2): track 2.91 -> 6.18 mm
- net Net-(D58-Pad2): track 2.91 -> 6.18 mm
- net Net-(D55-Pad2): track 2.91 -> 6.18 mm
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
Commit message: retrace, reorient, and all that
Parts:
- D1, D10, D11, D12, D13, D14, D15, D16, D17, D18, D19, D2, D20, D21, D22, D23, D24, D25, D26, D27, D28, D29, D3, D30, D31, D32, D33, D34, D35, D36, D37, D38, D39, D4, D40, D41, D42, D43, D44, D45, D46, D47, D48, D49, D5, D50, D51, D52, D53, D54, D55, D56, D57, D58, D59, D6, D60, D61, D62, D63, D64, D65, D66, D67, D68, D69, D7, D8, D9: moved to B.Cu
- SW1, SW10, SW11, SW12, SW13, SW14, SW15, SW16, SW17, SW18, SW19, SW2, SW20, SW21, SW22, SW23, SW24, SW25, SW26, SW27, SW28, SW29, SW3, SW30, SW31, SW32, SW33, SW34, SW35, SW36, SW37, SW38, SW39, SW4, SW40, SW41, SW42, SW43, SW44, SW45, SW46, SW47, SW48, SW49, SW5, SW50, SW51, SW52, SW53, SW54, SW55, SW56, SW57, SW58, SW59, SW6, SW60, SW61, SW62, SW63, SW64, SW65, SW66, SW67, SW68, SW69, SW7, SW8, SW9, U1: moved to F.Cu
- moved D69 7.95 mm to (358.9, 108.1)
- moved D67 7.56 mm to (318.9, 117.5), turned to 90 degrees
- moved D23 5.76 mm to (161.4, 127.3)
- moved D33 5.76 mm to (197.4, 127.3)
- moved D43 5.76 mm to (233.4, 127.3)
- moved D53 5.76 mm to (269.4, 127.3)
- moved D63 5.76 mm to (309.9, 127.3)
- moved D13 5.76 mm to (125.5, 127.3)
- moved D3 5.76 mm to (85.0, 127.3)
- moved D14 5.76 mm to (134.4, 144.3)
- moved D15 5.76 mm to (129.9, 161.3)
- moved D24 5.76 mm to (170.4, 144.3)
- moved D25 5.76 mm to (179.4, 161.3)
- moved D34 5.76 mm to (206.4, 144.3)
- moved D35 5.76 mm to (237.9, 161.3)
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Connections:
- U1 pad 10: R9 -> R0
- U1 pad 11: R8 -> R1
- U1 pad 12: R7 -> R2
- U1 pad 13: R6 -> R3
- U1 pad 14: R5 -> R4
- U1 pad 15: R4 -> R5
- U1 pad 16: R3 -> R6
- U1 pad 17: R2 -> R7
- U1 pad 18: R1 -> R8
- U1 pad 19: R0 -> R9
Routing:
- net R7: track 392.0 -> 291.4 mm
- net R5: track 360.1 -> 285.4 mm
- net R9: track 407.9 -> 336.0 mm
- net R1: track 314.6 -> 247.6 mm
- net R3: track 303.9 -> 243.1 mm
- net R8: track 376.7 -> 318.6 mm
- net C2: track 409.6 -> 370.3 mm
- net C6: track 226.0 -> 262.6 mm
- net R6: track 311.9 -> 275.6 mm
- net C5: track 298.4 -> 266.9 mm
- net C1: track 417.3 -> 388.4 mm
- net C3: track 357.7 -> 329.0 mm
- net R0: track 300.3 -> 272.9 mm
- net R4: track 287.5 -> 260.7 mm
- net C4: track 321.2 -> 294.8 mm
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Other:
- board size 305 x 86 mm -> 305 x 91.5 mm

Commit message: retrace front
Routing:
- net C3: track 329.0 -> 356.2 mm
- net C2: track 370.3 -> 391.7 mm
- net C1: track 388.4 -> 400.8 mm
- net C5: track 266.9 -> 278.6 mm
- net C4: track 294.8 -> 302.5 mm
- net C6: track 262.6 -> 257.6 mm
- net C0: track 433.1 -> 430.4 mm
