File: choc660/choc660.kicad_sch (KiCad schematic)
At the start: 137 parts, among them SW1 SW_Push, SW10 SW_Push, SW11 SW_Push, SW12 SW_Push, SW13 SW_Push, SW14 SW_Push, SW15 SW_Push, SW16 SW_Push, SW17 SW_Push, SW18 SW_Push, SW19 SW_Push, SW2 SW_Push, SW20 SW_Push, SW21 SW_Push, SW22 SW_Push, SW23 SW_Push, SW24 SW_Push, SW25 SW_Push, SW26 SW_Push, SW27 SW_Push, SW28 SW_Push, SW29 SW_Push, SW3 SW_Push, SW30 SW_Push, SW31 SW_Push, SW32 SW_Push, SW33 SW_Push, SW34 SW_Push, SW35 SW_Push, SW36 SW_Push, SW37 SW_Push, SW38 SW_Push, SW39 SW_Push, SW4 SW_Push, SW40 SW_Push, SW41 SW_Push, SW42 SW_Push, SW43 SW_Push, SW44 SW_Push, SW45 SW_Push, SW46 SW_Push, SW47 SW_Push, SW48 SW_Push, SW49 SW_Push, SW5 SW_Push, SW50 SW_Push, SW51 SW_Push, SW52 SW_Push, SW53 SW_Push, SW54 SW_Push, SW55 SW_Push, SW56 SW_Push, SW57 SW_Push, SW58 SW_Push, SW59 SW_Push, SW6 SW_Push, SW60 SW_Push, SW61 SW_Push, SW62 SW_Push, SW63 SW_Push, SW64 SW_Push, SW65 SW_Push, SW66 SW_Push, SW67 SW_Push, SW68 SW_Push, SW7 SW_Push, SW8 SW_Push, SW9 SW_Push, U1 Elite-C

Commit message: start work on placing footprints
Parts:
- added S1, S2, S3, S4, S5, S6, S7: MX_stab, marbastlib-choc:STAB_choc_2u, symbol marbastlib-mx:MX_stab
- SW62: footprint marbastlib-choc:SW_choc_HS_1.5u -> marbastlib-choc:SW_choc_HS_1u
Changed lines of the file:
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@@
     (property "Reference" "SW62" (id 0) (at 204.47 40.64 0))
     (property "Value" "SW_Push" (id 1) (at 204.47 43.18 0))
-    (property "Footprint" "marbastlib-choc:SW_choc_HS_1.5u" (id 2) (at 204.47 43.18 0)
+    (property "Footprint" "marbastlib-choc:SW_choc_HS_1u" (id 2) (at 204.47 43.18 0)
       (effects (font (size 1.27 1.27)) hide)
     )
@@
     (pin "2")
   )
+  (symbol (lib_id "marbastlib-mx:MX_stab") (at 104.14 160.02 0) (unit 1)
+    (in_bom yes) (on_board yes) (fields_autoplaced)
+    (property "Reference" "S3" (id 0) (at 110.49 158.6229 0)
+      (effects (font (size 1.27 1.27)) (justify left))
+    )
+    (property "Value" "MX_stab" (id 1) (at 110.49 161.1629 0)
+      (effects (font (size 1.27 1.27)) (justify left))
+    )
+    (property "Footprint" "marbastlib-choc:STAB_choc_2u" (id 2) (at 104.14 160.02 0)
+      (effects (font (size 1.27 1.27)) hide)
+    )
+    (property "Datasheet" "" (id 3) (at 104.14 160.02 0)
+      (effects (font (size 1.27 1.27)) hide)
+    )
+  )
   (symbol (lib_id "Switch:SW_Push") (at 162.56 29.21 0) (unit 1)
     (in_bom yes) (on_board yes) (fields_autoplaced)
@@
     (pin "2")
   )
+  (symbol (lib_id "marbastlib-mx:MX_stab") (at 104.14 144.78 0) (unit 1)
+    (in_bom yes) (on_board yes) (fields_autoplaced)
+    (property "Reference" "S1" (id 0) (at 110.49 143.3829 0)
+      (effects (font (size 1.27 1.27)) (justify left))
+    )
+    (property "Value" "MX_stab" (id 1) (at 110.49 145.9229 0)
+      (effects (font (size 1.27 1.27)) (justify left))
+    )
+    (property "Footprint" "marbastlib-choc:STAB_choc_2u" (id 2) (at 104.14 144.78 0)
+      (effects (font (size 1.27 1.27)) hide)
+    )
+    (property "Datasheet" "" (id 3) (at 104.14 144.78 0)
+      (effects (font (size 1.27 1.27)) hide)
+    )
+  )
   (symbol (lib_id "Switch:SW_Push") (at 50.8 48.26 0) (unit 1)
     (in_bom yes) (on_board yes) (fields_autoplaced)
@@
     (pin "2")
   )
+  (symbol (lib_id "marbastlib-mx:MX_stab") (at 104.14 167.64 0) (unit 1)
+    (in_bom yes) (on_board yes) (fields_autoplaced)
+    (property "Reference" "S4" (id 0) (at 110.49 166.2429 0)
+      (effects (font (size 1.27 1.27)) (justify left))
+    )
+    (property "Value" "MX_stab" (id 1) (at 110.49 168.7829 0)
+      (effects (font (size 1.27 1.27)) (justify left))
+    )
+    (property "Footprint" "marbastlib-choc:STAB_choc_2u" (id 2) (at 104.14 167.64 0)
+      (effects (font (size 1.27 1.27)) hide)
+    )
+    (property "Datasheet" "" (id 3) (at 104.14 167.64 0)
+      (effects (font (size 1.27 1.27)) hide)
+    )
+  )
   (symbol (lib_id "Device:D_Small") (at 45.72 54.61 90) (unit 1)
     (in_bom yes) (on_board yes) (fields_autoplaced)
@@
     (pin "2")
   )
+  (symbol (lib_id "marbastlib-mx:MX_stab") (at 124.46 144.78 0) (unit 1)
+    (in_bom yes) (on_board yes) (fields_autoplaced)
+    (property "Reference" "S5" (id 0) (at 130.81 143.3829 0)
+      (effects (font (size 1.27 1.27)) (justify left))
+    )
+    (property "Value" "MX_stab" (id 1) (at 130.81 145.9229 0)
+      (effects (font (size 1.27 1.27)) (justify left))
+    )
+    (property "Footprint" "marbastlib-choc:STAB_choc_2u" (id 2) (at 124.46 144.78 0)
+      (effects (font (size 1.27 1.27)) hide)
+    )
+    (property "Datasheet" "" (id 3) (at 124.46 144.78 0)
+      (effects (font (size 1.27 1.27)) hide)
+    )
+  )
   (symbol (lib_id "Switch:SW_Push") (at 78.74 107.95 0) (unit 1)
     (in_bom yes) (on_board yes) (fields_autoplaced)
@@
     (pin "2")
   )
+  (symbol (lib_id "marbastlib-mx:MX_stab") (at 124.46 160.02 0) (unit 1)
+    (in_bom yes) (on_board yes) (fields_autoplaced)
+    (property "Reference" "S7" (id 0) (at 130.81 158.6229 0)
+      (effects (font (size 1.27 1.27)) (justify left))
+    )
+    (property "Value" "MX_stab" (id 1) (at 130.81 161.1629 0)
+      (effects (font (size 1.27 1.27)) (justify left))
+    )
+    (property "Footprint" "marbastlib-choc:STAB_choc_2u" (id 2) (at 124.46 160.02 0)
+      (effects (font (size 1.27 1.27)) hide)
+    )
+    (property "Datasheet" "" (id 3) (at 124.46 160.02 0)
+      (effects (font (size 1.27 1.27)) hide)
+    )
+  )
   (symbol (lib_id "Switch:SW_Push") (at 120.65 88.9 0) (unit 1)
     (in_bom yes) (on_board yes) (fields_autoplaced)
@@
     (pin "2")
   )
+  (symbol (lib_id "marbastlib-mx:MX_stab") (at 104.14 152.4 0) (unit 1)
+    (in_bom yes) (on_board yes) (fields_autoplaced)
+    (property "Reference" "S2" (id 0) (at 110.49 151.0029 0)
+      (effects (font (size 1.27 1.27)) (justify left))
+    )
+    (property "Value" "MX_stab" (id 1) (at 110.49 153.5429 0)
+      (effects (font (size 1.27 1.27)) (justify left))
+    )
+    (property "Footprint" "marbastlib-choc:STAB_choc_2u" (id 2) (at 104.14 152.4 0)
+      (effects (font (size 1.27 1.27)) hide)
+    )
+    (property "Datasheet" "" (id 3) (at 104.14 152.4 0)
+      (effects (font (size 1.27 1.27)) hide)
+    )
+  )
   (symbol (lib_id "Device:D_Small") (at 199.39 95.25 90) (unit 1)
     (in_bom yes) (on_board yes) (fields_autoplaced)
@@
     (pin "1")
     (pin "2")
+  )
+  (symbol (lib_id "marbastlib-mx:MX_stab") (at 124.46 152.4 0) (unit 1)
+    (in_bom yes) (on_board yes) (fields_autoplaced)
+    (property "Reference" "S6" (id 0) (at 130.81 151.0029 0)
+      (effects (font (size 1.27 1.27)) (justify left))
+    )
+    (property "Value" "MX_stab" (id 1) (at 130.81 153.5429 0)
+      (effects (font (size 1.27 1.27)) (justify left))
+    )
+    (property "Footprint" "marbastlib-choc:STAB_choc_2u" (id 2) (at 124.46 152.4 0)
+      (effects (font (size 1.27 1.27)) hide)
+    )
+    (property "Datasheet" "" (id 3) (at 124.46 152.4 0)
+      (effects (font (size 1.27 1.27)) hide)
+    )
   )
   (symbol (lib_id "Switch:SW_Push") (at 64.77 68.58 0) (unit 1)
@@
       (reference "D68") (unit 1) (value "SOD-123") (footprint "Diode_SMD:D_SOD-123")
     )
+    (path "/64fa76e6-dba7-457e-9f62-1875288b3e4b"
+      (reference "S1") (unit 1) (value "MX_stab") (footprint "marbastlib-choc:STAB_choc_2u")
+    )
+    (path "/e1a089b4-c527-4687-aed3-c8bf3f8331d0"
+      (reference "S2") (unit 1) (value "MX_stab") (footprint "marbastlib-choc:STAB_choc_2u")
+    )
+    (path "/5b92b6be-e489-4cf1-b89c-dafa128f3ccf"
+      (reference "S3") (unit 1) (value "MX_stab") (footprint "marbastlib-choc:STAB_choc_2u")
+    )
+    (path "/7c23b365-bed0-4615-a188-25fffabab761"
+      (reference "S4") (unit 1) (value "MX_stab") (footprint "marbastlib-choc:STAB_choc_2u")
+    )
+    (path "/d12b765d-5873-4d8b-be7f-59e693a224d2"
+      (reference "S5") (unit 1) (value "MX_stab") (footprint "marbastlib-choc:STAB_choc_2u")
+    )
+    (path "/eb6a7a76-55de-4e79-a2be-634e2e7bd05c"
+      (reference "S6") (unit 1) (value "MX_stab") (footprint "marbastlib-choc:STAB_choc_2u")
+    )
+    (path "/dad23298-77f2-43ef-b06e-54db78125658"
+      (reference "S7") (unit 1) (value "MX_stab") (footprint "marbastlib-choc:STAB_choc_2u")
+    )
     (path "/630cd423-c8a1-4dea-9b7c-9a08c1a05824"
       (reference "SW1") (unit 1) (value "SW_Push") (footprint "marbastlib-choc:SW_choc_HS_1u")
@@
     )
     (path "/4736dc21-db65-4a2a-b797-607ccf4ab5b9"
-      (reference "SW62") (unit 1) (value "SW_Push") (footprint "marbastlib-choc:SW_choc_HS_1.5u")
+      (reference "SW62") (unit 1) (value "SW_Push") (footprint "marbastlib-choc:SW_choc_HS_1u")
     )
     (path "/c884e49f-49ee-4cd5-a146-e1f82b613be1"

Commit message: draw the rest of the owl?
Parts:
- removed S1, S2, S3, S4, S5, S6, S7: MX_stab, marbastlib-choc:STAB_choc_2u, symbol marbastlib-mx:MX_stab
- added D65: SOD-123, Diode_SMD:D_SOD-123, symbol Device:D_Small
- added SW65: SW_Push, marbastlib-choc:SW_choc_HS_1u, symbol Switch:SW_Push
- SW20, SW25, SW30, SW35, SW4, SW59, SW63: footprint marbastlib-choc:SW_choc_HS_1u -> marbastlib-choc:SW_choc_HS_1.5u
- SW66: renamed from SW65; footprint marbastlib-choc:SW_choc_HS_1u -> marbastlib-choc:SW_choc_HS_1.5u
- SW67: renamed from SW66; footprint marbastlib-choc:SW_choc_HS_1.5u -> marbastlib-choc:SW_choc_HS_1u
- renumbered D65 to D66, D66 to D67, D67 to D68, D68 to D69, SW67 to SW68, SW68 to SW69
Connections:
- net C6: now also SW65.2
- net R0: now also U1.19 (A2/PF5); no longer U1.10 (7/PE6)
- net R1: now also U1.18 (A1/PF6); no longer U1.11 (8/PB4)
- net R2: now also U1.17 (A0/PF7); no longer U1.12 (9/PB5)
- net R3: now also U1.16 (15/PB1); no longer U1.13 (10/PB6)
- net R4: now also U1.15 (14/PB3); no longer U1.14 (16/PB2)
- net R5: now also U1.14 (16/PB2); no longer U1.15 (14/PB3)
- net R6: now also U1.13 (10/PB6); no longer U1.16 (15/PB1)
- net R7: now also U1.12 (9/PB5); no longer U1.17 (A0/PF7)
- net R8: now also U1.11 (8/PB4), D65.1 (K); no longer U1.18 (A1/PF6)
- net R9: now also U1.10 (7/PE6); no longer U1.19 (A2/PF5)
- new net: D65.2 (A), SW65.1

Commit message: use non-hotswap footprints, also i made this backwards
Parts:
- SW1, SW10, SW11, SW12, SW13, SW14, SW15, SW16, SW17, SW18, SW19, SW21, SW22, SW23, SW24, SW26, SW27, SW28, SW29, SW31, SW32, SW33, SW34, SW36, SW37, SW38, SW39, SW40, SW41, SW42, SW43, SW44, SW45, SW46, SW47, SW48, SW49, SW5, SW50, SW51, SW52, SW53, SW54, SW55, SW56, SW57, SW58, SW6, SW60, SW61, SW62, SW64, SW65, SW67, SW68, SW69, SW7, SW8, SW9: footprint marbastlib-choc:SW_choc_HS_1u -> marbastlib-choc:SW_choc_1u
- SW2, SW25, SW3, SW30, SW35, SW4, SW59, SW63, SW66: footprint marbastlib-choc:SW_choc_HS_1.5u -> marbastlib-choc:SW_choc_1.5u
- SW20: footprint marbastlib-choc:SW_choc_HS_1.5u -> marbastlib-choc:SW_choc_1.25u

Commit message: retrace, reorient, and all that
Connections:
- net R0: now also U1.10 (7/PE6); no longer U1.19 (A2/PF5)
- net R1: now also U1.11 (8/PB4); no longer U1.18 (A1/PF6)
- net R2: now also U1.12 (9/PB5); no longer U1.17 (A0/PF7)
- net R3: now also U1.13 (10/PB6); no longer U1.16 (15/PB1)
- net R4: now also U1.14 (16/PB2); no longer U1.15 (14/PB3)
- net R5: now also U1.15 (14/PB3); no longer U1.14 (16/PB2)
- net R6: now also U1.16 (15/PB1); no longer U1.13 (10/PB6)
- net R7: now also U1.17 (A0/PF7); no longer U1.12 (9/PB5)
- net R8: now also U1.18 (A1/PF6); no longer U1.11 (8/PB4)
- net R9: now also U1.19 (A2/PF5); no longer U1.10 (7/PE6)
Changed lines of the file:
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@@
     )
   )
-  (global_label "R5" (shape input) (at 67.31 167.64 0) (fields_autoplaced)
+  (global_label "R4" (shape input) (at 67.31 167.64 0) (fields_autoplaced)
     (effects (font (size 1.27 1.27)) (justify left))
     (property "Intersheet References" "${INTERSHEET_REFS}" (id 0) (at 72.2026 167.5606 0)
@@
     )
   )
-  (global_label "R3" (shape input) (at 67.31 162.56 0) (fields_autoplaced)
+  (global_label "R6" (shape input) (at 67.31 162.56 0) (fields_autoplaced)
     (effects (font (size 1.27 1.27)) (justify left))
     (property "Intersheet References" "${INTERSHEET_REFS}" (id 0) (at 72.2026 162.4806 0)
@@
     )
   )
-  (global_label "R9" (shape input) (at 31.75 165.1 180) (fields_autoplaced)
+  (global_label "R0" (shape input) (at 31.75 165.1 180) (fields_autoplaced)
     (effects (font (size 1.27 1.27)) (justify right))
     (property "Intersheet References" "${INTERSHEET_REFS}" (id 0) (at 26.8574 165.0206 0)
@@
     )
   )
-  (global_label "R6" (shape input) (at 67.31 170.18 0) (fields_autoplaced)
+  (global_label "R3" (shape input) (at 67.31 170.18 0) (fields_autoplaced)
     (effects (font (size 1.27 1.27)) (justify left))
     (property "Intersheet References" "${INTERSHEET_REFS}" (id 0) (at 72.2026 170.1006 0)
@@
     )
   )
-  (global_label "R4" (shape input) (at 67.31 165.1 0) (fields_autoplaced)
+  (global_label "R5" (shape input) (at 67.31 165.1 0) (fields_autoplaced)
     (effects (font (size 1.27 1.27)) (justify left))
     (property "Intersheet References" "${INTERSHEET_REFS}" (id 0) (at 72.2026 165.0206 0)
@@
     )
   )
-  (global_label "R7" (shape input) (at 31.75 170.18 180) (fields_autoplaced)
+  (global_label "R2" (shape input) (at 31.75 170.18 180) (fields_autoplaced)
     (effects (font (size 1.27 1.27)) (justify right))
     (property "Intersheet References" "${INTERSHEET_REFS}" (id 0) (at 26.8574 170.1006 0)
@@
     )
   )
-  (global_label "R0" (shape input) (at 67.31 154.94 0) (fields_autoplaced)
+  (global_label "R9" (shape input) (at 67.31 154.94 0) (fields_autoplaced)
     (effects (font (size 1.27 1.27)) (justify left))
     (property "Intersheet References" "${INTERSHEET_REFS}" (id 0) (at 72.2026 154.8606 0)
@@
     )
   )
-  (global_label "R8" (shape input) (at 31.75 167.64 180) (fields_autoplaced)
+  (global_label "R1" (shape input) (at 31.75 167.64 180) (fields_autoplaced)
     (effects (font (size 1.27 1.27)) (justify right))
     (property "Intersheet References" "${INTERSHEET_REFS}" (id 0) (at 26.8574 167.5606 0)
@@
     )
   )
-  (global_label "R1" (shape input) (at 67.31 157.48 0) (fields_autoplaced)
+  (global_label "R8" (shape input) (at 67.31 157.48 0) (fields_autoplaced)
     (effects (font (size 1.27 1.27)) (justify left))
     (property "Intersheet References" "${INTERSHEET_REFS}" (id 0) (at 72.2026 157.4006 0)
@@
     )
   )
-  (global_label "R2" (shape input) (at 67.31 160.02 0) (fields_autoplaced)
+  (global_label "R7" (shape input) (at 67.31 160.02 0) (fields_autoplaced)
     (effects (font (size 1.27 1.27)) (justify left))
     (property "Intersheet References" "${INTERSHEET_REFS}" (id 0) (at 72.2026 159.9406 0)

Commit message: fix a footprint
Parts:
- SW20: footprint marbastlib-choc:SW_choc_1.25u -> marbastlib-choc:SW_choc_1.5u
Changed lines of the file:
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@@
     (property "Reference" "SW20" (id 0) (at 78.74 100.33 0))
     (property "Value" "SW_Push" (id 1) (at 78.74 102.87 0))
-    (property "Footprint" "marbastlib-choc:SW_choc_1.25u" (id 2) (at 78.74 102.87 0)
+    (property "Footprint" "marbastlib-choc:SW_choc_1.5u" (id 2) (at 78.74 102.87 0)
       (effects (font (size 1.27 1.27)) hide)
     )
@@
     )
     (path "/d14605ea-d48f-44ad-a2d7-845f3728e2f2"
-      (reference "SW20") (unit 1) (value "SW_Push") (footprint "marbastlib-choc:SW_choc_1.25u")
+      (reference "SW20") (unit 1) (value "SW_Push") (footprint "marbastlib-choc:SW_choc_1.5u")
     )
     (path "/769ec98f-af4d-4aaf-9ae9-776c0dad85f5"
