File: polo/polo/polo.kicad_pcb (KiCad board)
At the start: 2 copper layers, 58.7 x 39.7 mm, 25 parts, among them J1 Conn_01x04_MountingPin, Q1 AO3400A, SW1 SW_Push, SW2 SW_Push, SW3 SW_Push, SW4 SW_Push, SW5 SW_Push, SW6 SW_Push, U1 STM32F042F6Px, U2 XC6206P332MR

Commit message: update circuitboard with correct pin assignments lol
Parts:
- removed C13, C5, C6: 100nF, Capacitor_SMD:C_0805_2012Metric
- moved C9 35.2 mm to (148.4, 47.8), turned to 90 degrees
- moved C12 34.7 mm to (150.4, 51.2), turned to -90 degrees
- moved C3 32.3 mm to (150.4, 47.8), turned to 90 degrees
- moved C4 26.2 mm to (156.6, 44.2)
- moved R3 7.20 mm to (176.4, 45.8), turned to -90 degrees
- moved U2 5.41 mm to (145.3, 47.8), turned to 180 degrees
- moved C7 4.64 mm to (144.8, 42.2), turned to 0 degrees
- moved C8 3.61 mm to (144.8, 44.4), turned to 0 degrees
- moved U1 1.42 mm to (157.5, 49.0), turned to 180 degrees
Connections:
- U1 pad 11: D- -> unconnected-(U1-PA5-Pad11)
- U1 pad 12: D+ -> unconnected-(U1-PA6-Pad12)
- U1 pad 17: unconnected-(U1-PA9/PA11-Pad17) -> D-
- U1 pad 18: unconnected-(U1-PA10/PA12-Pad18) -> D+
Routing:
- net GND: track 134.9 -> 46.8 mm, vias 4 -> 5
- net +3.3V: track 98.0 -> 58.9 mm, vias 1 -> 2
- net RESET: track 27.9 -> 20.6 mm
- net X1: track 30.7 -> 36.8 mm
- net X3: track 29.3 -> 26.0 mm
- net Y1: track 19.5 -> 21.8 mm
- net Y3: track 21.4 -> 19.2 mm
- net +5V: track 13.5 -> 11.6 mm
- net D-: track 13.3 -> 15.1 mm
- net D+: track 13.3 -> 15.1 mm
- net X2: track 13.7 -> 13.0 mm
