File: polo/polo/polo.kicad_sch (KiCad schematic)
At the start: 25 parts, among them J1 Conn_01x04_MountingPin, Q1 AO3400A, SW1 SW_Push, SW2 SW_Push, SW3 SW_Push, SW4 SW_Push, SW5 SW_Push, SW6 SW_Push, U1 STM32F042F6Px, U2 XC6206P332MR

Commit message: update circuitboard with correct pin assignments lol
Parts:
- removed C13, C5, C6: 100nF, Capacitor_SMD:C_0805_2012Metric, symbol Device:C
Connections:
- net D+: now also U1.18 (PA10/PA12); no longer U1.12 (PA6)
- net D-: now also U1.17 (PA9/PA11); no longer U1.11 (PA5)
Other:
- moved on the sheet: C12
